File: Rain_Gauge/V1.5/EDA/RainGauge_PCB.kicad_pcb (KiCad board)
At the start: 2 copper layers, 64 x 40.5 mm, 13 parts, among them Q1 2N2219, U1 DS3231M, U2 SD_Card, U3 Battery_Leads, U4 Electrode_TH, U5 Electrode_TH

Commit message: Reorganize and new PCB
Parts:
- added BT1: Battery, ARTS-Lab:battery_holder_10mm, F.Cu at (129.5, 95.2)
- added G***: LOGO, ARTS-Lab:uofsc_logo_0_75in, B.Cu at (124.0, 113.8)
- moved U3 17.5 mm to (141.0, 88.9), turned to 0 degrees
- moved Q1 5.08 mm to (159.2, 95.7)
- moved S1 5.08 mm to (146.6, 93.5), turned to 270 degrees
- renumbered R1 to 3M1
Connections:
- 3M1 pad 1: Net-(A1-Pad19) -> Net-(3M1-Pad1)
- A1 pad 1: (no net) -> Net-(A1-Pad1)
- A1 pad 10: (no net) -> Net-(A1-Pad10)
- A1 pad 11: (no net) -> Net-(A1-Pad11)
- A1 pad 12: (no net) -> Net-(A1-Pad12)
- A1 pad 13: (no net) -> Net-(A1-Pad13)
- A1 pad 18: (no net) -> Net-(A1-Pad18)
- A1 pad 19: Net-(A1-Pad19) -> Net-(3M1-Pad1)
- A1 pad 2: (no net) -> Net-(A1-Pad2)
- A1 pad 20: (no net) -> Net-(A1-Pad20)
- A1 pad 21: (no net) -> Net-(A1-Pad21)
- A1 pad 22: (no net) -> Net-(A1-Pad22)
- A1 pad 25: (no net) -> Net-(A1-Pad25)
- A1 pad 26: (no net) -> Net-(A1-Pad26)
- A1 pad 28: (no net) -> Net-(A1-Pad28)
- A1 pad 3: (no net) -> Net-(A1-Pad3)
- A1 pad 6: (no net) -> Net-(A1-Pad6)
- A1 pad 8: (no net) -> Net-(A1-Pad8)
- A1 pad 9: (no net) -> Net-(A1-Pad9)
- U1 pad 1: (no net) -> Net-(U1-Pad1)
- U1 pad 14: (no net) -> Net-(BT1-Pad1)
- U1 pad 4: (no net) -> Net-(U1-Pad4)
Routing:
- net Net-(BT1-Pad1): track 0.00 -> 31.7 mm
- net Net-(A1-Pad19): track 23.3 -> 0.00 mm
- net Net-(3M1-Pad1): track 0.00 -> 15.2 mm
- net Net-(S1-Pad2): track 19.4 -> 10.4 mm
- net Net-(Q1-Pad2): track 27.0 -> 21.9 mm
- net Net-(A1-Pad27): track 40.7 -> 37.7 mm
- net Net-(A1-Pad30): track 11.1 -> 10.3 mm
- net Net-(10k1-Pad2): track 72.8 -> 72.9 mm, vias 4 -> 6

Commit message: KiCad Stuff
Parts:
- moved 4.7k1 5.85 mm to (122.5, 119.0)
- moved 4.7k2 0.71 mm to (131.5, 125.0), turned to 90 degrees
- turned C1 to 90 degrees
Routing:
- net Net-(10k1-Pad1): track 77.3 -> 70.2 mm
- net Net-(4.7k1-Pad2): track 54.8 -> 49.9 mm
- net Net-(10k1-Pad2): track 72.9 -> 69.7 mm, vias 6 -> 2
- net Net-(3M1-Pad1): track 15.2 -> 12.0 mm
- net Net-(4.7k2-Pad2): track 34.7 -> 35.7 mm
