File: Rain_Gauge/V1.5/EDA/RainGauge_PCB.sch (KiCad schematic (older format))
At the start: 13 parts

Commit message: KiCad Stuff
Parts:
- added BT1: Battery, ARTS-Lab:battery_holder_10mm, symbol Device:Battery
- 10k1: renamed from 10k; footprint (none) -> Resistor_SMD:R_0201_0603Metric_Pad0.64x0.40mm_HandSolder
- 3M1: renamed from 3M; footprint (none) -> Resistor_SMD:R_0201_0603Metric_Pad0.64x0.40mm_HandSolder
- 4.7k1, 4.7k2: renamed from 4.7k; footprint (none) -> Resistor_SMD:R_0201_0603Metric_Pad0.64x0.40mm_HandSolder
- C1: renamed from C?; footprint (none) -> Capacitor_SMD:C_0201_0603Metric_Pad0.64x0.40mm_HandSolder
- U2: renamed from U?; footprint (none) -> Project-lib:SD_card
- U3: renamed from U?; footprint (none) -> Project-lib:battery_leads
- U4, U5: renamed from U?; footprint (none) -> Project-lib:electrode
- gave numbers to parts that had none: 4
Connections:
- wire segments 58 -> 60
Changed lines of the file:
@@
 $EndDescr
 $Comp
-L MCU_Module:Arduino_Nano_v3.x A?
+L MCU_Module:Arduino_Nano_v3.x A1
 U 1 1 6205BC37
 P 5500 4000
-F 0 "A?" V 5600 3850 50  0000 C CNN
+F 0 "A1" V 5600 3850 50  0000 C CNN
 F 1 "Arduino_Nano_v3.x" V 5500 3900 50  0000 C CNN
 F 2 "Module:Arduino_Nano" H 5500 4000 50  0001 C CIN
@@
 $EndComp
 $Comp
-L RainGauge_PCB-rescue:Electrode_TH-Schematics U?
+L RainGauge_PCB-rescue:Electrode_TH-Schematics U4
 U 1 1 6205DB53
 P 7700 2900
-F 0 "U?" V 7475 3037 50  0000 C CNN
+F 0 "U4" V 7475 3037 50  0000 C CNN
 F 1 "Electrode_TH" V 7566 3037 50  0000 C CNN
-F 2 "" H 7700 2900 50  0001 C CNN
+F 2 "Project-lib:electrode" H 7700 2900 50  0001 C CNN
 F 3 "" H 7700 2900 50  0001 C CNN
 	1    7700 2900
@@
 $EndComp
 $Comp
-L RainGauge_PCB-rescue:SD_Card-Schematics U?
+L RainGauge_PCB-rescue:SD_Card-Schematics U2
 U 1 1 6205E3A1
 P 4250 4900
-F 0 "U?" H 3900 5050 50  0000 R CNN
+F 0 "U2" H 3900 5050 50  0000 R CNN
 F 1 "SD_Card" H 3900 5150 50  0000 R CNN
-F 2 "" H 4250 4900 50  0001 C CNN
+F 2 "Project-lib:SD_card" H 4250 4900 50  0001 C CNN
 F 3 "" H 4250 4900 50  0001 C CNN
 	1    4250 4900
@@
 $EndComp
 $Comp
-L Device:R 4.7k
+L Device:R 4.7k1
 U 1 1 620605D5
 P 3500 3650
-F 0 "4.7k" H 3250 3700 50  0000 L CNN
+F 0 "4.7k1" H 3250 3700 50  0000 L CNN
 F 1 "R" H 3350 3600 50  0000 L CNN
-F 2 "" V 3430 3650 50  0001 C CNN
+F 2 "Resistor_SMD:R_0201_0603Metric_Pad0.64x0.40mm_HandSolder" V 3430 3650 50  0001 C CNN
 F 3 "~" H 3500 3650 50  0001 C CNN
 	1    3500 3650
@@
 $EndComp
 $Comp
-L Device:R 10k
+L Device:R 10k1
 U 1 1 62060AD0
 P 3500 3400
-F 0 "10k" H 3600 3450 50  0000 L CNN
+F 0 "10k1" H 3600 3450 50  0000 L CNN
 F 1 "R" H 3570 3355 50  0000 L CNN
-F 2 "" V 3430 3400 50  0001 C CNN
+F 2 "Resistor_SMD:R_0201_0603Metric_Pad0.64x0.40mm_HandSolder" V 3430 3400 50  0001 C CNN
 F 3 "~" H 3500 3400 50  0001 C CNN
 	1    3500 3400
@@
 $EndComp
 $Comp
-L Device:R 3M
+L Device:R 3M1
 U 1 1 62060D30
 P 7050 4150
-F 0 "3M" H 7120 4196 50  0000 L CNN
+F 0 "3M1" H 7120 4196 50  0000 L CNN
 F 1 "R" H 7120 4105 50  0000 L CNN
-F 2 "" V 6980 4150 50  0001 C CNN
+F 2 "Resistor_SMD:R_0201_0603Metric_Pad0.64x0.40mm_HandSolder" V 6980 4150 50  0001 C CNN
 F 3 "~" H 7050 4150 50  0001 C CNN
 	1    7050 4150
@@
 $EndComp
 $Comp
-L Device:R 4.7k
+L Device:R 4.7k2
 U 1 1 620610FA
 P 4600 2150
-F 0 "4.7k" H 4670 2196 50  0000 L CNN
+F 0 "4.7k2" H 4670 2196 50  0000 L CNN
 F 1 "R" H 4670 2105 50  0000 L CNN
-F 2 "" V 4530 2150 50  0001 C CNN
+F 2 "Resistor_SMD:R_0201_0603Metric_Pad0.64x0.40mm_HandSolder" V 4530 2150 50  0001 C CNN
 F 3 "~" H 4600 2150 50  0001 C CNN
 	1    4600 2150
@@
 $EndComp
 $Comp
-L power:GND #PWR?
+L power:GND #PWR0101
 U 1 1 6206211D
 P 6350 2100
-F 0 "#PWR?" H 6350 1850 50  0001 C CNN
+F 0 "#PWR0101" H 6350 1850 50  0001 C CNN
 F 1 "GND" H 6355 1927 50  0000 C CNN
 F 2 "" H 6350 2100 50  0001 C CNN
@@
 $EndComp
 $Comp
-L RainGauge_PCB-rescue:EG1218-dk_Slide-Switches S?
+L RainGauge_PCB-rescue:EG1218-dk_Slide-Switches S1
 U 1 1 62063322
 P 6250 2300
-F 0 "S?" V 6204 2444 50  0000 L CNN
+F 0 "S1" V 6204 2444 50  0000 L CNN
 F 1 "EG1218" V 6295 2444 50  0000 L CNN
 F 2 "digikey-footprints:Switch_Slide_11.6x4mm_EG1218" H 6450 2500 50  0001 L CNN
@@
 $EndComp
 $Comp
-L RainGauge_PCB-rescue:Battery_Leads-Schematics U?
+L RainGauge_PCB-rescue:Battery_Leads-Schematics U3
 U 1 1 62067DF3
 P 6300 1900
-F 0 "U?" H 6478 1913 50  0000 L CNN
+F 0 "U3" H 6478 1913 50  0000 L CNN
 F 1 "Battery_Leads" H 6478 1822 50  0000 L CNN
-F 2 "" H 6300 1900 50  0001 C CNN
+F 2 "Project-lib:battery_leads" H 6300 1900 50  0001 C CNN
 F 3 "" H 6300 1900 50  0001 C CNN
 	1    6300 1900
@@
 $EndComp
 $Comp
-L Timer_RTC:DS3231M U?
+L Timer_RTC:DS3231M U1
 U 1 1 62068A2D
 P 3900 2650
-F 0 "U?" H 4200 2300 50  0000 C CNN
+F 0 "U1" H 4200 2300 50  0000 C CNN
 F 1 "DS3231M" H 3600 2300 50  0000 C CNN
 F 2 "Package_SO:SOIC-16W_7.5x10.3mm_P1.27mm" H 3900 2050 50  0001 C CNN
@@
 $EndComp
 $Comp
-L power:GND #PWR?
+L power:GND #PWR0102
 U 1 1 620732FA
 P 6350 2500
-F 0 "#PWR?" H 6350 2250 50  0001 C CNN
+F 0 "#PWR0102" H 6350 2250 50  0001 C CNN
 F 1 "GND" H 6355 2327 50  0000 C CNN
 F 2 "" H 6350 2500 50  0001 C CNN
@@
 $EndComp
 $Comp
-L power:GND #PWR?
+L power:GND #PWR0103
 U 1 1 62073943
 P 4500 4800
-F 0 "#PWR?" H 4500 4550 50  0001 C CNN
+F 0 "#PWR0103" H 4500 4550 50  0001 C CNN
 F 1 "GND" H 4505 4627 50  0000 C CNN
 F 2 "" H 4500 4800 50  0001 C CNN
@@
 $EndComp
 $Comp
-L Device:C C?
+L Device:C C1
 U 1 1 6207284C
 P 4900 2100
-F 0 "C?" H 5015 2146 50  0000 L CNN
+F 0 "C1" H 5015 2146 50  0000 L CNN
 F 1 "C" H 5015 2055 50  0000 L CNN
-F 2 "" H 4938 1950 50  0001 C CNN
+F 2 "Capacitor_SMD:C_0201_0603Metric_Pad0.64x0.40mm_HandSolder" H 4938 1950 50  0001 C CNN
 F 3 "~" H 4900 2100 50  0001 C CNN
 	1    4900 2100
@@
 	4900 2250 4900 2350
 $Comp
-L power:GND #PWR?
+L power:GND #PWR0104
 U 1 1 62089C83
 P 4900 2350
-F 0 "#PWR?" H 4900 2100 50  0001 C CNN
+F 0 "#PWR0104" H 4900 2100 50  0001 C CNN
 F 1 "GND" H 4905 2177 50  0000 C CNN
 F 2 "" H 4900 2350 50  0001 C CNN
@@
 	4800 4500 5000 4500
 $Comp
-L power:GND #PWR?
+L power:GND #PWR0105
 U 1 1 62094AFE
 P 5500 5000
-F 0 "#PWR?" H 5500 4750 50  0001 C CNN
+F 0 "#PWR0105" H 5500 4750 50  0001 C CNN
 F 1 "GND" H 5505 4827 50  0000 C CNN
 F 2 "" H 5500 5000 50  0001 C CNN
@@
 $EndComp
 $Comp
-L power:GND #PWR?
+L power:GND #PWR0106
 U 1 1 62094F84
 P 5600 5000
-F 0 "#PWR?" H 5600 4750 50  0001 C CNN
+F 0 "#PWR0106" H 5600 4750 50  0001 C CNN
 F 1 "GND" H 5605 4827 50  0000 C CNN
 F 2 "" H 5600 5000 50  0001 C CNN
@@
 $EndComp
 $Comp
-L power:GND #PWR?
+L power:GND #PWR0107
 U 1 1 620950E6
 P 4300 2650
-F 0 "#PWR?" H 4300 2400 50  0001 C CNN
+F 0 "#PWR0107" H 4300 2400 50  0001 C CNN
 F 1 "GND" V 4305 2522 50  0000 R CNN
 F 2 "" H 4300 2650 50  0001 C CNN
@@
 	5400 2750 5400 3000
 $Comp
-L power:GND #PWR?
+L power:GND #PWR0108
 U 1 1 62097FBB
 P 7050 4300
-F 0 "#PWR?" H 7050 4050 50  0001 C CNN
+F 0 "#PWR0108" H 7050 4050 50  0001 C CNN
 F 1 "GND" H 7055 4127 50  0000 C CNN
 F 2 "" H 7050 4300 50  0001 C CNN
@@
 	5700 2900 7050 2900
 $Comp
-L RainGauge_PCB-rescue:Electrode_TH-Schematics U?
+L RainGauge_PCB-rescue:Electrode_TH-Schematics U5
 U 1 1 6205EADF
 P 7700 3250
-F 0 "U?" V 7475 3387 50  0000 C CNN
+F 0 "U5" V 7475 3387 50  0000 C CNN
 F 1 "Electrode_TH" V 7566 3387 50  0000 C CNN
-F 2 "" H 7700 3250 50  0001 C CNN
+F 2 "Project-lib:electrode" H 7700 3250 50  0001 C CNN
 F 3 "" H 7700 3250 50  0001 C CNN
 	1    7700 3250
@@
 $EndComp
 $Comp
-L Transistor_BJT:2N2219 Q?
+L Transistor_BJT:2N2219 Q1
 U 1 1 620D90AA
 P 7150 3250
-F 0 "Q?" H 7341 3296 50  0000 L CNN
+F 0 "Q1" H 7341 3296 50  0000 L CNN
 F 1 "2N2219" H 7341 3205 50  0000 L CNN
 F 2 "Package_TO_SOT_THT:TO-39-3" H 7350 3175 50  0001 L CIN
@@
 	7050 4000 6000 4000
 Connection ~ 7050 4000
+$Comp
+L Device:Battery BT1
+U 1 1 6216EAAD
+P 2650 3150
+F 0 "BT1" H 2758 3196 50  0000 L CNN
+F 1 "Battery" H 2758 3105 50  0000 L CNN
+F 2 "ARTS-Lab:battery_holder_10mm" V 2650 3210 50  0001 C CNN
+F 3 "~" V 2650 3210 50  0001 C CNN
+	1    2650 3150
+	1    0    0    -1
+$EndComp
+Wire Wire Line
+	2650 2950 2650 2650
+Wire Wire Line
+	2650 2650 3500 2650
+$Comp
+L power:GND #PWR0109
+U 1 1 6217073B
+P 2650 3350
+F 0 "#PWR0109" H 2650 3100 50  0001 C CNN
+F 1 "GND" H 2655 3177 50  0000 C CNN
+F 2 "" H 2650 3350 50  0001 C CNN
+F 3 "" H 2650 3350 50  0001 C CNN
+	1    2650 3350
+	1    0    0    -1
+$EndComp
 $EndSCHEMATC
